Commit message: change : robot link in correctd 'frame is rotated at 180' in config xml file map update rate is corrected

File: my_robot/urdf/rrRobot.xacro (robot description, xacro)
@@ -162,5 +162,5 @@
     <parent link="robot_base"/>
     <child link="robot_back_support"/>
-    <origin rpy="0  0  0" xyz="0    -0.27   0.475"/>
+    <origin rpy="0  0  0" xyz="0    0.27   0.475"/>
     <axis xyz="0  0  0"/>
     <limit effort="0" lower="0" upper="0" velocity="0"/>
@@ -214,31 +214,31 @@
     <parent link="robot_base"/>
     <child link="front_caster"/>
+    <origin rpy="0  0  0" xyz="0     -0.245   -0.118"/>
+    <axis xyz="0  0  0"/>
+    <limit effort="0" lower="0" upper="0" velocity="0"/>
+  </joint>
+  <link name="back_caster">
+    <inertial>
+      <mass value="0.1"/>
+      <origin rpy="0  0  0" xyz="0  0  0"/>
+      <inertia ixx="0.1" ixy="0" ixz="0" iyy="0.1" iyz="0" izz="0.1"/>
+    </inertial>
+    <collision name="back_caster_collision">
+      <origin rpy="0  0  0" xyz="0  0  0"/>
+      <geometry>
+        <sphere radius="0.0605"/>
+      </geometry>
+    </collision>
+    <visual name="back_caster_visual">
+      <origin rpy="0  0  0" xyz="0  0  0"/>
+      <geometry>
+        <sphere radius="0.0605"/>
+      </geometry>
+    </visual>
+  </link>
+  <joint name="robot_base_back_caster" type="fixed">
+    <parent link="robot_base"/>
+    <child link="back_caster"/>
     <origin rpy="0  0  0" xyz="0     0.245   -0.118"/>
-    <axis xyz="0  0  0"/>
-    <limit effort="0" lower="0" upper="0" velocity="0"/>
-  </joint>
-  <link name="back_caster">
-    <inertial>
-      <mass value="0.1"/>
-      <origin rpy="0  0  0" xyz="0  0  0"/>
-      <inertia ixx="0.1" ixy="0" ixz="0" iyy="0.1" iyz="0" izz="0.1"/>
-    </inertial>
-    <collision name="back_caster_collision">
-      <origin rpy="0  0  0" xyz="0  0  0"/>
-      <geometry>
-        <sphere radius="0.0605"/>
-      </geometry>
-    </collision>
-    <visual name="back_caster_visual">
-      <origin rpy="0  0  0" xyz="0  0  0"/>
-      <geometry>
-        <sphere radius="0.0605"/>
-      </geometry>
-    </visual>
-  </link>
-  <joint name="robot_base_back_caster" type="fixed">
-    <parent link="robot_base"/>
-    <child link="back_caster"/>
-    <origin rpy="0  0  0" xyz="0     -0.245   -0.118"/>
     <axis xyz="0  0  0"/>
     <limit effort="0" lower="0" upper="0" velocity="0"/>
@@ -335,5 +335,5 @@
   </link>
   <joint type="fixed" name="camera_joint">
-    <origin xyz="0.0 0.285 0.060" rpy="0 0 1.5707"/>
+    <origin xyz="0.0 -0.285 0.060" rpy="0 0 -1.5707"/>
     <child link="camera"/>
     <parent link="robot_base"/>

Commit message: new: RTAB node + RGDB camera

File: my_robot/urdf/rrRobot.xacro (robot description, xacro)
@@ -340,4 +340,11 @@
     <axis xyz="1 0 0" rpy="0 0 0"/>
   </joint>
+  <link name="camera_link_optical">
+  </link>
+  <joint name="camera_optical_joint" type="fixed">
+    <origin xyz="0.0 -0.285 0.060" rpy="-1.5707 0 -1.5707"/>
+    <parent link="camera"/>
+    <child link="camera_link_optical"/>
+  </joint>
    <gazebo reference='left_wheel'>
        <material>Gazebo/Red</material>
